File: hardware/TMP006 Breakout.sch (EAGLE design)
At the start: 14 parts, among them U1 TMP006

Commit message: Added Fiducials to the board and paneled it
Parts:
- added FID1, FID2: FIDUCIALUFIDUCIAL, SparkFun-Aesthetics:FIDUCIALUFIDUCIAL
Changed lines of the file:
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@@
 <?xml version="1.0" encoding="utf-8"?>
 <!DOCTYPE eagle SYSTEM "eagle.dtd">
-<eagle version="6.2">
+<eagle version="6.5.0">
 <drawing>
 <settings>
@@
 <part name="STANDOFF2" library="SparkFun-Electromechanical" deviceset="STAND-OFF" device=""/>
 <part name="LOGO3" library="SparkFun-Aesthetics" deviceset="LOGO-SFE" device="NEW"/>
+<part name="FID1" library="SparkFun-Aesthetics" deviceset="FIDUCIAL" device="UFIDUCIAL"/>
+<part name="FID2" library="SparkFun-Aesthetics" deviceset="FIDUCIAL" device="UFIDUCIAL"/>
 </parts>
 <sheets>
@@
 <instance part="STANDOFF2" gate="G$1" x="238.76" y="17.78"/>
 <instance part="LOGO3" gate="G$1" x="231.14" y="25.4"/>
+<instance part="FID1" gate="G$1" x="154.94" y="38.1"/>
+<instance part="FID2" gate="G$1" x="162.56" y="38.1"/>
 </instances>
 <busses>
